File: ChromeOSServoAdapter.kicad_pcb (KiCad board)
At the start: 2 copper layers, 65 x 69.5 mm, 69 parts, among them J1 Raspberry_Pi_2_3, J10 Conn_01x01_Female, J11 Conn_01x01_Female, J12 Conn_01x01_Female, J13 Conn_01x01_Female, J2 Conn_01x08_Female, J3 Conn_01x02_Female, J4 Conn_02x25_Odd_Even, J5 Conn_02x03_Odd_Even, J6 Conn_02x03_Odd_Even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

Commit message: board intermediate
Parts:
- removed J10, J11, J9: Conn_01x01_Female, Connector_PinSocket_2.54mm:PinSocket_1x01_P2.54mm_Vertical
- moved C6 61.5 mm to (108.3, 82.8), turned to 0 degrees
- moved C4 59.3 mm to (108.3, 84.5), turned to 0 degrees
- moved U6 52.2 mm to (106.9, 90.1), turned to 270 degrees
- moved C5 50.8 mm to (111.5, 89.9), turned to 90 degrees
- moved C19 0.66 mm to (139.8, 93.2)
Routing:
- net VCC: track 21.8 -> 274.0 mm, vias 0 -> 1
- net Net-(J6-Pad4): track 0.00 -> 105.0 mm, vias 0 -> 2
- net /PPDUT_UART2_VREF: track 0.00 -> 103.6 mm, vias 0 -> 5
- net /1v8: track 15.5 -> 115.1 mm, vias 0 -> 2
- net /PPDUT_SPI2_VREF: track 0.00 -> 98.9 mm
- net Net-(C11-Pad1): track 2.66 -> 101.4 mm, vias 0 -> 1
- net /PPDUT_UART1_VREF: track 4.51 -> 99.0 mm, vias 0 -> 2
- net Net-(J1-Pad28): track 0.00 -> 77.7 mm, vias 0 -> 2
- net /DUT_GOOG_REC_MODE_L: track 0.00 -> 77.3 mm, vias 0 -> 3
- net /KBD_COL1: track 0.00 -> 74.6 mm, vias 0 -> 1
- net Net-(J1-Pad40): track 0.00 -> 73.2 mm, vias 0 -> 2
- net /PPDUT_SPI1_VREF: track 7.87 -> 81.0 mm, vias 0 -> 3
- net Net-(J1-Pad24): track 1.94 -> 73.9 mm, vias 1 -> 4
- net /DUT_JTAG_TDI_BUF: track 0.00 -> 71.4 mm, vias 0 -> 6
- net GND: track 137.4 -> 208.6 mm
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Other:
- net class power: clearance 0.2 -> 0.19

Commit message: board production ready
Parts:
- added G***: LOGO, ChromeOSServoAdapter:license, F.Cu at (160.2, 75.5)
- added J9: Conn_01x01_Female, ChromeOSServoAdapter:S1x1, F.Cu at (106.7, 111.8)
- D3, D4: footprint LED_THT:LED_D3.0mm -> ChromeOSServoAdapter:LED_D3mm
- J12, J13: footprint Connector_PinSocket_2.54mm:PinSocket_1x01_P2.54mm_Vertical -> ChromeOSServoAdapter:S1x1
- J2: footprint Connector_PinSocket_2.54mm:PinSocket_1x08_P2.54mm_Vertical -> ChromeOSServoAdapter:S1x8
- J3: footprint Connector_PinSocket_2.54mm:PinSocket_1x02_P2.54mm_Vertical -> ChromeOSServoAdapter:S1x2
- J5, J6: footprint Connector_PinSocket_2.54mm:PinSocket_2x03_P2.54mm_Vertical -> ChromeOSServoAdapter:S2x3
- JP2, JP3, JP4: footprint Connector_PinSocket_2.54mm:PinSocket_1x03_P2.54mm_Vertical -> ChromeOSServoAdapter:JP3
- moved C3 11.9 mm to (124.6, 74.7), turned to 0 degrees
- moved C2 9.88 mm to (142.2, 76.0), turned to 180 degrees
- moved C7 8.88 mm to (139.4, 82.3), turned to 270 degrees
- moved C19 0.40 mm to (139.4, 93.2)
- moved R5 0.06 mm to (124.5, 108.8)
- turned C11 to 180 degrees
- turned C23 to 0 degrees
Connections:
- C25 pad 1: Net-(C25-Pad1) -> /PPDUT_UART2_VREF
- C9 pad 1: Net-(C25-Pad1) -> Net-(C9-Pad1)
- JP3 pad 2: Net-(C25-Pad1) -> Net-(C9-Pad1)
- U7 pad 1: Net-(C25-Pad1) -> Net-(C9-Pad1)
- U7 pad 14: Net-(C25-Pad1) -> Net-(C9-Pad1)
Routing:
- net GND: track 208.6 -> 610.1 mm, vias 0 -> 26
- net /JTAG_TMS: track 0.00 -> 94.2 mm, vias 0 -> 5
- net Net-(C9-Pad1): track 0.00 -> 72.9 mm, vias 0 -> 2
- net Net-(C25-Pad1): track 61.2 -> 0.00 mm, vias 1 -> 0
- net Net-(J1-Pad38): track 1.47 -> 61.6 mm, vias 1 -> 2
- net Net-(J1-Pad23): track 2.08 -> 57.0 mm, vias 1 -> 4
- net Net-(JP2-Pad2): track 64.8 -> 22.4 mm, vias 5 -> 0
- net /DUT_COLD_RESET_L: track 0.00 -> 36.8 mm, vias 0 -> 4
- net Net-(J1-Pad11): track 1.64 -> 35.2 mm, vias 1 -> 4
- net VCC: track 274.0 -> 300.7 mm, vias 1 -> 6
- net /HPD: track 0.00 -> 23.3 mm
- net /1v8: track 115.1 -> 138.1 mm
- net /PPDUT_UART1_VREF: track 99.0 -> 111.5 mm
- net /DUT_PWR_BUTTON: track 36.3 -> 48.7 mm
- net Net-(J1-Pad28): track 77.7 -> 88.8 mm
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- added copper zone on B.Cu, net GND
Other:
- board text added: "ChromeOSServoAdapter - Back"
